File: SDX_gerbers/Stradex1.kicad_sch (KiCad schematic)
At the start: 24 parts, among them SW1 SW_Push, SW2 SW_Push, SW3 SW_Push, SW4 SW_Push, U1 ADS1115IDGS, U2 ADS1115IDGS

Commit message: modified a few things
Other:
- note added: "Analogue to digital converterc (ADC's)"
- note added: "Buttons (String indicators)"
- note added: "Microcontroller"
- note added: "Potentiomeeters"
- note added: "SoftPot"
- moved on the sheet: R1, R10, R11, R12, R17, R2, R3, R4, R5, R6, R7, R8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
