File: PCB/Stradex1.kicad_pcb (KiCad board)
At the start: 4 copper layers, 192.1 x 126.9 mm, 24 parts, among them SW1 SW_Push, SW2 SW_Push, SW3 SW_Push, SW4 SW_Push, U1 ADS1115IDGS, U2 ADS1115IDGS

Commit message: Made the pcb 2 layers and added a gnd copper fill
Parts:
- moved R12 11.9 mm to (90.7, 133.0)
- moved R8 11.2 mm to (90.7, 139.5)
Routing:
- net GND: track 651.5 -> 0.00 mm
- net +3.3V: track 604.6 -> 436.1 mm
- net /SCL: track 103.8 -> 34.9 mm
- net /FSR3: track 183.7 -> 115.1 mm
- net /PB1: track 110.4 -> 46.6 mm
- net /PB2: track 121.2 -> 59.3 mm
- net /FSR4: track 172.8 -> 138.1 mm, vias 0 -> 6
- net /P1: track 89.7 -> 56.9 mm
- net /SDA: track 106.3 -> 89.3 mm
- net /SPot: track 143.2 -> 126.8 mm
- net /ALRT1: track 35.8 -> 25.2 mm
- net /FSR1: track 69.1 -> 58.8 mm
- net /PB3: track 107.6 -> 98.3 mm
- net /P2: track 44.9 -> 35.9 mm
- net /PB4: track 132.9 -> 124.6 mm, vias 0 -> 2
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- added copper zone on B.Cu, net GND
- added copper zone on F.Cu, net GND
Other:
- copper layers 4 -> 2

Commit message: Stole the pcb from 'Whitebowfr'
Parts:
- added R13: 10k, Resistor_THT:R_Axial_DIN0207_L6.3mm_D2.5mm_P7.62mm_Horizontal, F.Cu at (201.8, 36.0)
- added SW5: MT_JUMPER_1, Jumper:SolderJumper-3_P1.3mm_Open_RoundedPad1.0x1.5mm, F.Cu at (209.3, 40.1)
- added SW6: MT_JUMPER_1, Jumper:SolderJumper-3_P1.3mm_Open_RoundedPad1.0x1.5mm, F.Cu at (206.0, 40.1)
- added SW7: MT_JUMPER_1, Jumper:SolderJumper-3_P1.3mm_Open_RoundedPad1.0x1.5mm, F.Cu at (212.6, 40.1)
- moved R8 92.9 mm to (174.9, 100.2), turned to 180 degrees
- moved R12 81.3 mm to (172.0, 132.8), turned to -90 degrees
- moved R7 67.4 mm to (174.9, 96.7), turned to 180 degrees
- moved R9 58.5 mm to (157.2, 132.7), turned to -90 degrees
- moved R11 44.8 mm to (167.5, 132.7), turned to -90 degrees
- moved R10 44.1 mm to (162.5, 132.7), turned to -90 degrees
- moved R17 27.3 mm to (194.2, 39.2)
- moved R5 18.3 mm to (174.9, 89.8), turned to 180 degrees
- moved R6 16.6 mm to (174.9, 93.3), turned to 180 degrees
Connections:
- A1 pad 31: unconnected-(A1-GPIO26_ADC0-Pad31) -> /SPot_MT
- R17 pad 1: /SPot -> GND
- R17 pad 2: GND -> /SPot
- RV1 pad 1: /SPot -> Net-(SW7-B)
- RV1 pad 2: +3.3V -> Net-(SW5-B)
- RV1 pad 3: GND -> Net-(SW6-B)
Routing:
- net /SPot_MT: track 0.00 -> 149.2 mm, vias 0 -> 1
- net +3.3V: track 436.1 -> 301.6 mm, vias 0 -> 3
- net GND: track 0.00 -> 122.4 mm, vias 0 -> 211
- net /PB1: track 46.6 -> 106.9 mm
- net /SCL: track 34.9 -> 83.8 mm
- net Net-(SW6-B): track 0.00 -> 28.9 mm
- net /PB2: track 59.3 -> 85.0 mm
- net Net-(SW5-B): track 0.00 -> 24.7 mm
- net Net-(SW7-B): track 0.00 -> 18.9 mm
- net /SPot: track 126.8 -> 110.2 mm, vias 0 -> 2
- net /P3: track 44.1 -> 59.5 mm
- net /P1: track 56.9 -> 71.0 mm
- net /FSR1: track 58.8 -> 69.1 mm
- net /PB4: track 124.6 -> 132.7 mm, vias 2 -> 0
- net /ALRT2: track 47.0 -> 55.1 mm
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Other:
- board text added: "Multi touch"
- board text added: "Single touch"
