File: PCB/Stradex1.kicad_sch (KiCad schematic)
At the start: 24 parts, among them SW1 SW_Push, SW2 SW_Push, SW3 SW_Push, SW4 SW_Push, U1 ADS1115IDGS, U2 ADS1115IDGS

Commit message: Stole the pcb from 'Whitebowfr'
Parts:
- removed R1, R2, R3, R4: FSR, Connector_PinSocket_2.54mm:PinSocket_1x02_P2.54mm_Vertical, symbol My_Parts:FSR
- added R1, R2, R3, R4: FSR, Connector_PinSocket_2.54mm:PinSocket_1x02_P2.54mm_Vertical, symbol Device:R_Variable
- added R13, R14, R15: 10k, Resistor_THT:R_Axial_DIN0207_L6.3mm_D2.5mm_P7.62mm_Horizontal, symbol Device:R
- added RV5, RV6: SoftPot, Connector_PinSocket_2.54mm:PinSocket_1x03_P2.54mm_Vertical, symbol My_Parts:SoftPot
- added SW5, SW6, SW7: MT_JUMPER_1, Jumper:SolderJumper-3_P1.3mm_Open_RoundedPad1.0x1.5mm, symbol Switch:SW_SPDT
Connections:
- net +3.3V: now also RV5.1, RV6.2, SW5.3 (C), SW7.1 (A); no longer RV1.2
- net FSR1: now also R1.2
- net FSR2: now also R2.2
- net FSR3: now also R3.2
- net FSR4: now also R4.2
- net GND: now also R17.1, R1.1, R13.2, R14.1, R15.2, R2.1, R3.1, R4.1, RV5.3, SW6.1 (A); no longer R17.2, RV1.3
- net SPot: now also R17.2, R14.2, RV5.2, RV6.3, SW5.1 (A), SW6.3 (C); no longer R17.1, RV1.1
- net SPot_MT: now reaches A1.31 (GPIO26_ADC0)
- net SPot_MT: now also R13.1, R15.1, RV6.1, SW7.3 (C)
- new net: RV1.1, SW7.2 (B)
- new net: RV1.2, SW5.2 (B)
- new net: RV1.3, SW6.2 (B)
- no-connect marks 0 -> 22
Other:
- note removed: "Analogue to digital converterc (ADC's)"
- note removed: "Buttons (String indicators)"
- note removed: "Microcontroller"
- note removed: "Potentiomeeters"
- note removed: "SoftPot"
- moved on the sheet: R10, R11, R12, R17, R5, R6, R7, R8, R9, RV1, RV2, RV3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
